Commit message: catkin pt.4 TODO needs correctly scaled stl

File: src/toaster-description/urdf/toaster.urdf.xacro (robot description, xacro)
@@ -1,4 +1,4 @@
-<?<?xml version="1.0"?>
-<<robot name="toaster xmlns:xacro="http://www.ros.org/wiki/xacro">
+<?xml version="1.0"?>
+<robot name="toaster" xmlns:xacro="http://www.ros.org/wiki/xacro">
     <xacro:property name="PI" value="3.1415926535897932" />
     <xacro:property name="wheelbase" value="0.400" />
@@ -60,8 +60,8 @@
     </xacro:macro>
     <xacro:wheel prefix="left">
-        <origin xyz="${wheelbase/2} 0 ${wheel_vertical_offset}" rpy="0 0 0" />
+        <origin xyz="0.200 0 ${wheel_vertical_offset}" rpy="0 0 0" />
     </xacro:wheel>
     <xacro:wheel prefix="right">
-        <origin xyz="$-{wheelbase/2} 0 ${wheel_vertical_offset}" rpy="0 0 0" />
+        <origin xyz="-0.200 0 ${wheel_vertical_offset}" rpy="0 0 0" />
     </xacro:wheel>
     <link name="base_link"></link>
@@ -107,4 +107,4 @@
     </link>
       <!-- Bring in simulation data for Gazebo. -->
-    <xacro:include filename="$(find toaster_description)/urdf/toaster.gazebo" />
+    <xacro:include filename="$(find toaster-description)/urdf/toaster.gazebo" />
 </robot>

Commit message: Changed scale of stl

File: src/toaster-description/urdf/toaster.urdf.xacro (robot description, xacro)
@@ -15,5 +15,5 @@
                 <origin xyz="0 0 0" rpy="${PI/2} 0 0"/>
                 <geometry>
-                    <mesh filename="package://toaster-description/meshes/toaster-wheel.stl"/>
+                    <mesh filename="package://toaster-description/meshes/toaster-wheel.stl" scale="0.001 0.001 0.001"/>
                 </geometry>
                 <material name="black" />
@@ -85,5 +85,5 @@
         <origin xyz="0 0 0" rpy="0 0 0"/>
         <geometry>
-            <mesh filename="package://toaster-description/meshes/toaster-chassis.stl"/>
+            <mesh filename="package://toaster-description/meshes/toaster-chassis.stl" scale="0.001 0.001 0.001"/>
         </geometry>
             <material name="dark_grey" />
@@ -92,5 +92,5 @@
             <origin xyz="0 0 0" rpy="0 0 0"/>
             <geometry>
-                <mesh filename="package://toaster-description/meshes/toaster-chassis.stl"/>
+                <mesh filename="package://toaster-description/meshes/toaster-chassis.stl" scale="0.001 0.001 0.001"/>
             </geometry>
         </collision>

Commit message: Added casters

File: src/toaster-description/urdf/toaster.urdf.xacro (robot description, xacro)
@@ -35,5 +35,5 @@
         </link>
         <gazebo reference="${prefix}_wheel_link">
-            <material>Gazebo/DarkGrey</material>
+            <material>Gazebo/Black</material>
             <selfCollide>false</selfCollide>
             <mu1 value="0.5"/>
@@ -60,8 +60,8 @@
     </xacro:macro>
     <xacro:wheel prefix="left">
-        <origin xyz="0.200 0 ${wheel_vertical_offset}" rpy="0 0 0" />
+        <origin xyz="0 0.2 ${wheel_vertical_offset}" rpy="0 0 0" />
     </xacro:wheel>
     <xacro:wheel prefix="right">
-        <origin xyz="-0.200 0 ${wheel_vertical_offset}" rpy="0 0 0" />
+        <origin xyz="0 -0.2 ${wheel_vertical_offset}" rpy="0 0 0" />
     </xacro:wheel>
     <link name="base_link"></link>
@@ -106,4 +106,56 @@
         </inertial>
     </link>
+    <!--Caster front  -->
+  <link name="caster_front_link">
+    <visual>
+      <origin rpy="1.57079632679 0 0" xyz="0 0 0"/>
+      <geometry>
+        <sphere radius="0.02"/>
+      </geometry>
+      <material name="Black"/>
+    </visual>
+    <collision>
+      <geometry>
+        <sphere radius="0.02"/>
+      </geometry>
+      <origin rpy="1.57079632679 0 0" xyz="0 0 0"/>
+    </collision>
+    <inertial>
+      <mass value="0.5"/>
+      <origin xyz="0 0 0"/>
+      <inertia ixx="0.001" ixy="0.0" ixz="0.0" iyy="0.001" iyz="0.0" izz="0.001"/>
+    </inertial>
+  </link>
+  <joint name="caster_front_joint" type="fixed">
+    <parent link="base_link"/>
+    <child link="caster_front_link"/>
+    <origin rpy="-1.57079632679 0 0" xyz="0.2032 0.0 -0.127"/>
+  </joint>
+  <!--Caster back  -->
+  <link name="caster_back_link">
+    <visual>
+      <origin rpy="1.57079632679 0 0" xyz="0.0 0.0 0 "/>
+      <geometry>
+        <sphere radius="0.02"/>
+      </geometry>
+      <material name="Black"/>
+    </visual>
+    <collision>
+      <geometry>
+        <sphere radius="0.02"/>
+      </geometry>
+      <origin rpy="1.57079632679 0 0" xyz="0 0.0 0 "/>
+    </collision>
+    <inertial>
+      <mass value="0.5"/>
+      <origin xyz="0 0 0"/>
+      <inertia ixx="0.001" ixy="0.0" ixz="0.0" iyy="0.001" iyz="0.0" izz="0.001"/>
+    </inertial>
+  </link>
+  <joint name="caster_back_joint" type="fixed">
+    <parent link="base_link"/>
+    <child link="caster_back_link"/>
+    <origin rpy="-1.57079632679 0 0" xyz="-0.2032 0.0 -.127"/>
+  </joint>
       <!-- Bring in simulation data for Gazebo. -->
     <xacro:include filename="$(find toaster-description)/urdf/toaster.gazebo" />

Commit message: remove error

File: src/toaster-description/urdf/toaster.urdf.xacro (robot description, xacro)
@@ -71,5 +71,5 @@
         <child link="chassis_link" />
     </joint>
-    git <link name="imu_link">
+    <link name="imu_link">
         <inertial>
         <mass value="0.001"/>

Commit message: added move base and gmapping

File: src/toaster-description/urdf/toaster.urdf.xacro (robot description, xacro)
@@ -133,29 +133,55 @@
   </joint>
   <!--Caster back  -->
-  <link name="caster_back_link">
-    <visual>
-      <origin rpy="1.57079632679 0 0" xyz="0.0 0.0 0 "/>
-      <geometry>
-        <sphere radius="0.02"/>
-      </geometry>
-      <material name="Black"/>
-    </visual>
-    <collision>
-      <geometry>
-        <sphere radius="0.02"/>
-      </geometry>
-      <origin rpy="1.57079632679 0 0" xyz="0 0.0 0 "/>
-    </collision>
-    <inertial>
-      <mass value="0.5"/>
-      <origin xyz="0 0 0"/>
-      <inertia ixx="0.001" ixy="0.0" ixz="0.0" iyy="0.001" iyz="0.0" izz="0.001"/>
-    </inertial>
+    <link name="caster_back_link">
+        <visual>
+        <origin rpy="1.57079632679 0 0" xyz="0.0 0.0 0 "/>
+        <geometry>
+            <sphere radius="0.02"/>
+        </geometry>
+        <material name="Black"/>
+        </visual>
+        <collision>
+        <geometry>
+            <sphere radius="0.02"/>
+        </geometry>
+        <origin rpy="1.57079632679 0 0" xyz="0 0.0 0 "/>
+        </collision>
+        <inertial>
+        <mass value="0.5"/>
+        <origin xyz="0 0 0"/>
+        <inertia ixx="0.001" ixy="0.0" ixz="0.0" iyy="0.001" iyz="0.0" izz="0.001"/>
+        </inertial>
+    </link>
+    <joint name="caster_back_joint" type="fixed">
+        <parent link="base_link"/>
+        <child link="caster_back_link"/>
+        <origin rpy="-1.57079632679 0 0" xyz="-0.2032 0.0 -.127"/>
+    </joint>
+    <joint name="hokuyo_joint" type="fixed">
+        <axis xyz="0 1 0" />
+        <origin xyz="0 0 .25" rpy="0 0 0"/>
+        <parent link="base_link"/>
+        <child link="hokuyo_link"/>
+  </joint>
+  <!-- Hokuyo Laser -->
+    <link name="hokuyo_link">
+        <collision>
+            <origin xyz="0 0 0" rpy="0 0 0"/>
+            <geometry>
+                <box size="0.1 0.1 0.1"/>
+            </geometry>
+        </collision>
+        <visual>
+            <origin xyz="0 0 0" rpy="0 0 0"/>
+                <geometry>
+                    <sphere radius="0.02"/>
+                </geometry>
+        </visual>
+        <inertial>
+            <mass value="1e-5" />
+            <origin xyz="0 0 0" rpy="0 0 0"/>
+            <inertia ixx="1e-6" ixy="0" ixz="0" iyy="1e-6" iyz="0" izz="1e-6" />
+        </inertial>
   </link>
-  <joint name="caster_back_joint" type="fixed">
-    <parent link="base_link"/>
-    <child link="caster_back_link"/>
-    <origin rpy="-1.57079632679 0 0" xyz="-0.2032 0.0 -.127"/>
-  </joint>
       <!-- Bring in simulation data for Gazebo. -->
     <xacro:include filename="$(find toaster-description)/urdf/toaster.gazebo" />

Commit message: wip fix laser

File: src/toaster-description/urdf/toaster.urdf.xacro (robot description, xacro)
@@ -160,5 +160,5 @@
     <joint name="hokuyo_joint" type="fixed">
         <axis xyz="0 1 0" />
-        <origin xyz="0 0 .25" rpy="0 0 0"/>
+        <origin xyz="0 0 0" rpy="0 0 0"/>
         <parent link="base_link"/>
         <child link="hokuyo_link"/>

Commit message: lidar fix wip

File: src/toaster-description/urdf/toaster.urdf.xacro (robot description, xacro)
@@ -158,12 +158,12 @@
         <origin rpy="-1.57079632679 0 0" xyz="-0.2032 0.0 -.127"/>
     </joint>
-    <joint name="hokuyo_joint" type="fixed">
+    <!-- Laser -->
+    <joint name="laser_joint" type="fixed">
         <axis xyz="0 1 0" />
         <origin xyz="0 0 .25" rpy="0 0 0"/>
         <parent link="base_link"/>
-        <child link="hokuyo_link"/>
+        <child link="laser_link"/>
   </joint>
-  <!-- Hokuyo Laser -->
-    <link name="hokuyo_link">
+    <link name="laser_link">
         <collision>
             <origin xyz="0 0 0" rpy="0 0 0"/>

Commit message: few name changes

File: src/toaster-description/urdf/toaster.urdf.xacro (robot description, xacro)
@@ -161,5 +161,5 @@
     <joint name="laser_joint" type="fixed">
         <axis xyz="0 1 0" />
-        <origin xyz="0 0 0" rpy="0 0 0"/>
+        <origin xyz="0 0 0.25" rpy="0 0 0"/>
         <parent link="base_link"/>
         <child link="laser_link"/>

Commit message: config changes

File: src/toaster-description/urdf/toaster.urdf.xacro (robot description, xacro)
@@ -2,5 +2,5 @@
 <robot name="toaster" xmlns:xacro="http://www.ros.org/wiki/xacro">
     <xacro:property name="PI" value="3.1415926535897932" />
-    <xacro:property name="wheelbase" value="0.400" />
+    <xacro:property name="wheelbase" value="0.550" />
     <xacro:property name="wheel_radius" value="0.125" />
     <xacro:property name="wheel_width" value="0.100" />
@@ -60,8 +60,8 @@
     </xacro:macro>
     <xacro:wheel prefix="left">
-        <origin xyz="0 0.2 ${wheel_vertical_offset}" rpy="0 0 0" />
+        <origin xyz="0 0.24 ${wheel_vertical_offset}" rpy="0 0 0" />
     </xacro:wheel>
     <xacro:wheel prefix="right">
-        <origin xyz="0 -0.2 ${wheel_vertical_offset}" rpy="0 0 0" />
+        <origin xyz="0 -0.24 ${wheel_vertical_offset}" rpy="0 0 0" />
     </xacro:wheel>
     <link name="base_link"></link>
@@ -130,5 +130,5 @@
     <parent link="base_link"/>
     <child link="caster_front_link"/>
-    <origin rpy="-1.57079632679 0 0" xyz="0.2032 0.0 -0.127"/>
+    <origin rpy="-1.57079632679 0 0" xyz="0.2032 0.0 -0.128"/>
   </joint>
   <!--Caster back  -->
